File: hackdeck.kicad_pcb (KiCad board)
At the start: 2 copper layers, 76.2 x 83.8 mm, 13 parts, among them SW1 SW_Push, SW2 SW_Push, SW3 SW_Push, SW4 SW_Push, SW5 RotaryEncoder, SW6 SW_Push, SW7 SW_Push, U1 XIAO-RP2040-DIP, U2 OLED

Commit message: final stretch
Parts:
- turned D3 to 0 degrees
- turned D4 to 0 degrees
Routing:
- net +5V: track 0.00 -> 327.0 mm
- net GND: track 0.00 -> 247.2 mm
- net Net-(U1-GPIO26/ADC0/A0): track 0.00 -> 128.9 mm
- net Net-(D2-DOUT): track 0.00 -> 73.7 mm
- net Net-(U1-GPIO28/ADC2/A2): track 0.00 -> 73.1 mm
- net Net-(U1-GPIO7/SCL): track 0.00 -> 65.7 mm
- net Net-(D1-DOUT): track 0.00 -> 65.2 mm
- net Net-(D3-DOUT): track 0.00 -> 63.9 mm
- net Net-(U1-GPIO6/SDA): track 0.00 -> 58.4 mm
- net Net-(U1-GPIO0/TX): track 0.00 -> 52.8 mm
- net Net-(U1-GPIO27/ADC1/A1): track 0.00 -> 46.0 mm
- net Net-(U1-GPIO29/ADC3/A3): track 0.00 -> 39.9 mm
- net Net-(U1-GPIO1/RX): track 0.00 -> 33.8 mm
- net Net-(D1-DIN): track 0.00 -> 30.1 mm
- net Net-(U1-GPIO4/MISO): track 0.00 -> 19.1 mm
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Other:
- board text added: "XIAO HERE"
- board text added: "ZENNIX HACKDECK"
