File: PCB/hackdeck.kicad_pcb (KiCad board)
At the start: 2 copper layers, 76.2 x 83.8 mm, 13 parts, among them SW1 SW_Push, SW2 SW_Push, SW3 SW_Push, SW4 SW_Push, SW5 RotaryEncoder, SW6 SW_Push, SW7 SW_Push, U1 XIAO-RP2040-DIP, U2 OLED

Commit message: OLED and Rotary fix
Routing:
- net Net-(U1-GPIO0/TX): track 52.8 -> 44.2 mm
- net Net-(U1-GPIO7/SCL): track 65.7 -> 61.0 mm
- net Net-(U1-GPIO6/SDA): track 58.4 -> 56.4 mm
Changed lines of the file:
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@@
 	)
 	(segment
-		(start 76.2 72.0725)
-		(end 76.2 107.15625)
+		(start 76.74525 104.5265)
+		(end 79.21625 106.9975)
 		(width 0.2)
 		(layer "F.Cu")
@@
 	(segment
 		(start 61.9125 57.785)
-		(end 76.2 72.0725)
+		(end 76.74525 72.61775)
 		(width 0.2)
 		(layer "F.Cu")
@@
 	)
 	(segment
-		(start 76.35875 106.9975)
-		(end 79.21625 106.9975)
-		(width 0.2)
-		(layer "F.Cu")
-		(net 11)
-	)
-	(segment
-		(start 76.2 107.15625)
-		(end 76.35875 106.9975)
+		(start 76.74525 72.61775)
+		(end 76.74525 104.5265)
 		(width 0.2)
 		(layer "F.Cu")
@@
 	)
 	(segment
-		(start 59.53125 62.70625)
-		(end 59.53125 80.9625)
+		(start 59.53125 78.58125)
+		(end 60.36875 77.74375)
 		(width 0.2)
 		(layer "B.Cu")
@@
 	)
 	(segment
-		(start 100.0125 80.9625)
-		(end 100.0125 78.69)
-		(width 0.2)
-		(layer "B.Cu")
-		(net 17)
-	)
-	(segment
-		(start 59.53125 80.9625)
-		(end 100.0125 80.9625)
-		(width 0.2)
-		(layer "B.Cu")
-		(net 17)
-	)
-	(segment
-		(start 100.0125 78.69)
+		(start 60.36875 77.74375)
 		(end 100.95875 77.74375)
 		(width 0.2)
@@
 	)
 	(segment
-		(start 99.9625 76.2)
+		(start 59.53125 62.70625)
+		(end 59.53125 78.58125)
+		(width 0.2)
+		(layer "B.Cu")
+		(net 17)
+	)
+	(segment
+		(start 74.25125 75.20375)
 		(end 100.95875 75.20375)
 		(width 0.2)
@@
 	)
 	(segment
-		(start 61.9125 76.2)
-		(end 99.9625 76.2)
+		(start 61.9125 62.865)
+		(end 74.25125 75.20375)
 		(width 0.2)
 		(layer "B.Cu")
-		(net 18)
-	)
-	(segment
-		(start 61.9125 62.865)
-		(end 61.9125 76.2)
-		(width 0.2)
-		(layer "B.Cu")
